File: Hardware/Qwiic_Chirp_101.sch (EAGLE design)
At the start: 31 parts, among them J1 QWIIC_RIGHT_ANGLE, J2 QWIIC_RIGHT_ANGLE, Q1 20V/0.2A/8MHz/1.2Ω/1Vth, Q2 20V/0.2A/8MHz/1.2Ω/1Vth, Q3 20V/0.2A/8MHz/1.2Ω/1Vth, Q6 20V/0.2A/8MHz/1.2Ω/1Vth, Q8 20V/0.2A/8MHz/1.2Ω/1Vth, U1 AP2127K-1.8V

Commit message: Cleaning up schematic
Other:
- note added: "0.1" Headers"
- note added: "FFC Connector"
- note added: "Logic-Level Conversion"
- note added: "Power LED"
- note added: "Qwiic Connectors"
- note added: "Voltage Regulator"
- moved on the sheet: C1, C2, D1, J1, J2, J4, J5, JP2, JP4, Q1, Q2, Q3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
